File: CM4_NAS.kicad_sch (KiCad schematic)
At the start: 30 parts, among them J1 USB_A, J10 Conn_02x07_Odd_Even, J11 Conn_01x03, J13 USB_OTG, J14 USB_select_jmpr, J15 Temp_Sensor, J2 HDMI_header, J3 PCIe_conn, J4 Sata_PWR, J5 PWR_IN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

Commit message: Fixed wrong footprint
Parts:
- U6: footprint Package_SO:SOIC-8_5.275x5.275mm_P1.27mm -> Package_SO:MSOP-8_3x3mm_P0.65mm
Changed lines of the file:
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@@
   (junction (at 275.59 109.22) (diameter 1.016) (color 0 0 0 0))
   (junction (at 275.59 111.76) (diameter 1.016) (color 0 0 0 0))
-  (no_connect (at 52.07 298.45))
-  (no_connect (at 182.88 130.81))
+  (no_connect (at 113.03 311.15))
+  (no_connect (at 139.7 186.69))
   (no_connect (at 44.45 33.02))
+  (no_connect (at 52.07 303.53))
+  (no_connect (at 52.07 308.61))
+  (no_connect (at 113.03 242.57))
+  (no_connect (at 271.78 106.68))
+  (no_connect (at 242.57 132.08))
   (no_connect (at 242.57 101.6))
-  (no_connect (at 113.03 311.15))
   (no_connect (at 52.07 306.07))
+  (no_connect (at 242.57 318.77))
+  (no_connect (at 242.57 116.84))
+  (no_connect (at 182.88 130.81))
+  (no_connect (at 52.07 298.45))
   (no_connect (at 242.57 316.23))
-  (no_connect (at 271.78 91.44))
   (no_connect (at 242.57 104.14))
-  (no_connect (at 52.07 308.61))
-  (no_connect (at 52.07 303.53))
+  (no_connect (at 271.78 91.44))
   (no_connect (at 44.45 30.48))
-  (no_connect (at 242.57 318.77))
-  (no_connect (at 242.57 132.08))
-  (no_connect (at 271.78 106.68))
-  (no_connect (at 242.57 116.84))
-  (no_connect (at 139.7 186.69))
-  (no_connect (at 113.03 242.57))
   (wire (pts (xy 27.94 76.2) (xy 44.45 76.2))
     (stroke (width 0) (type solid) (color 0 0 0 0))
@@
     (property "Reference" "U6" (id 0) (at 233.045 309.499 0))
     (property "Value" "EMC2301-1-ACZL-TR" (id 1) (at 233.045 311.8104 0))
-    (property "Footprint" "Package_SO:SOIC-8_5.275x5.275mm_P1.27mm" (id 2) (at 234.95 326.39 0)
+    (property "Footprint" "Package_SO:MSOP-8_3x3mm_P0.65mm" (id 2) (at 234.95 326.39 0)
       (effects (font (size 1.27 1.27)) hide)
     )
@@
     )
     (path "/806aaaa1-1057-4d4d-a02b-a9a49f02ddbb"
-      (reference "U6") (unit 1) (value "EMC2301-1-ACZL-TR") (footprint "Package_SO:SOIC-8_5.275x5.275mm_P1.27mm")
+      (reference "U6") (unit 1) (value "EMC2301-1-ACZL-TR") (footprint "Package_SO:MSOP-8_3x3mm_P0.65mm")
     )
   )

Commit message: new usb select header
Parts:
- removed J13: USB_OTG, Connector_PinSocket_2.54mm:PinSocket_1x05_P2.54mm_Vertical, symbol Connector:USB_OTG
- removed J14: USB_select_jmpr, Connector_PinHeader_2.54mm:PinHeader_2x03_P2.54mm_Vertical, symbol Connector_Generic:Conn_02x03_Odd_Even
- removed TP1: TestPoint, TestPoint:TestPoint_Pad_2.0x2.0mm, symbol Connector:TestPoint
- added J12: Conn_01x03, Connector_PinHeader_2.54mm:PinHeader_1x03_P2.54mm_Vertical, symbol Connector_Generic:Conn_01x03
Connections:
- net Master_USB2_N is gone; now on net USB2_N: J1.2 (D-)
- net Master_USB2_P is gone; now on net USB2_P: J1.3 (D+)
- net Slave_MicroUSB_N is gone; now on net USB2_N: U5.5 (D2-), U5.6
- net Slave_MicroUSB_P is gone; now on net USB2_P: U5.4 (D2+), U5.7
- net +5V: now also J12.1 (Pin_1); no longer J1.1 (VBUS)
- net USBOTG_ID: now also J12.3 (Pin_3)
- new net USB2_VBUS: J1.1 (VBUS), J12.2 (Pin_2)
- no-connect marks 18 -> 17
Other:
- note added: "The same connector is used for slave and master USB operation. Use a jumper to link the USB Vbus to the 5V rail for master operation. Use a jumper to link the USB Vbus to the USBOTG pin for slave operation."
- note added: "USB ESD protection"
- note removed: "Micro USB ESD protection"
- note removed: "Use two jumpers to choose which USB is routed to the CM4. Route the micro USB port to program eMMC. Route the USB type A to use slave devices with the CM4."
- moved on the sheet: U5

Commit message: HDMI, silkscreen, gpios...
Parts:
- added D2: LED Red, LED_THT:LED_D5.0mm, symbol Device:LED
- added J13: Conn_02x06_Odd_Even, Connector_PinHeader_2.54mm:PinHeader_2x06_P2.54mm_Vertical, symbol Connector_Generic:Conn_02x06_Odd_Even
- added R6: 1k, Resistor_THT:R_Axial_DIN0207_L6.3mm_D2.5mm_P7.62mm_Horizontal, symbol Device:R
- added U7: 74LVC1G07SE-7, Package_TO_SOT_SMD:SOT-353_SC-70-5, symbol CM4IO:74LVC1G07_copy
- J2: footprint CM4:PinSocket_2x10_P2.54mm_Vertical_alternate-pinout -> CM4:HDMI EDAC 690-019-298-412
Connections:
- net +3.3v: now also D2.2 (A), J13.10 (Pin_10), U7.5 (VCC)
- net +5V: now also J13.12 (Pin_12)
- net GND: now also J13.11 (Pin_11), U7.3 (GND)
- net GPIO12: now also J13.9 (Pin_9)
- net GPIO14: now also J13.7 (Pin_7)
- net GPIO15: now also J13.2 (Pin_2)
- net GPIO18: now also J13.4 (Pin_4)
- net GPIO2: now also J13.5 (Pin_5)
- net GPIO23: now also J13.6 (Pin_6)
- net GPIO24: now also J13.8 (Pin_8)
- net GPIO26: now also J13.1 (Pin_1)
- net GPIO3: now also J13.3 (Pin_3)
- net PCIE_RX_N: now also J3.A17 (PERN0); no longer J3.A16 (PERP0)
- net PCIE_RX_P: now also J3.A16 (PERP0); no longer J3.A17 (PERN0)
- net PCIE_TX_N: now also J3.B15 (PETN0); no longer J3.B14 (PETP0)
- net PCIE_TX_P: now also J3.B14 (PETP0); no longer J3.B15 (PETN0)
- net nPWR_LED: now also U7.2
- new net: R6.2, U7.4
- new net: D2.1 (K), R6.1
Other:
- note added: "PWR LED"
- note removed: "TX and RX have PN swaps to improve routing"

Commit message: rev1.4 Add pin to OLED connector for button, use SMD caps and LEDs, more info on silkscreen and fixed some traces.
Parts:
- removed J8: OLED_conn, Connector_JST:JST_XH_B4B-XH-A_1x04_P2.50mm_Vertical, symbol Connector_Generic:Conn_01x04
- added J8: OLED_conn, Connector_JST:JST_XH_B5B-XH-A_1x05_P2.50mm_Vertical, symbol Connector_Generic:Conn_01x05
- C1, C2: footprint Capacitor_THT:CP_Radial_D4.0mm_P2.00mm -> Capacitor_SMD:C_0805_2012Metric_Pad1.18x1.45mm_HandSolder
- D1, D2: footprint LED_THT:LED_D5.0mm -> LED_SMD:LED_0805_2012Metric_Pad1.15x1.40mm_HandSolder
Connections:
- net +3.3v: now also J8.4 (Pin_4)
- net GND: now also J8.5 (Pin_5)
- net SCL: now also J8.3 (Pin_3)
- net SDA: now also J8.2 (Pin_2)
- net GPIO7 renamed OLED_BTN
- net OLED_BTN: now also J8.1 (Pin_1)
Changed lines of the file:
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@@
     (stroke (width 0) (type solid) (color 0 0 0 0))
   )
+  (wire (pts (xy 27.94 365.76) (xy 38.1 365.76))
+    (stroke (width 0) (type solid) (color 0 0 0 0))
+  )
   (wire (pts (xy 27.94 368.3) (xy 38.1 368.3))
     (stroke (width 0) (type solid) (color 0 0 0 0))
@@
   )
   (text "I2C connection to external 128x32 OLED display.\nWould show the NAS status as well as relevant info\nsuch as IP address, temperatures, etc."
-    (at 68.58 367.03 0)
+    (at 68.58 363.22 0)
     (effects (font (size 1.27 1.27)) (justify right bottom))
   )
@@
     (effects (font (size 1.27 1.27)) (justify left bottom))
   )
+  (label "OLED_BTN" (at 27.94 365.76 180)
+    (effects (font (size 1.27 1.27)) (justify right bottom))
+  )
   (label "SDA" (at 27.94 368.3 180)
     (effects (font (size 1.27 1.27)) (justify right bottom))
@@
     (effects (font (size 1.27 1.27)) (justify right bottom))
   )
-  (label "GPIO7" (at 121.92 265.43 180)
-    (effects (font (size 1.27 1.27)) (justify right bottom))
-  )
   (label "GPIO8" (at 121.92 267.97 180)
     (effects (font (size 1.27 1.27)) (justify right bottom))
@@
     (effects (font (size 1.27 1.27)) (justify right bottom))
   )
+  (label "OLED_BTN" (at 127 265.43 0)
+    (effects (font (size 1.27 1.27)) (justify left bottom))
+  )
   (label "GLOBAL_EN" (at 127 344.17 180)
     (effects (font (size 1.27 1.27)) (justify right bottom))
@@
       (effects (font (size 1.27 1.27)) (justify right))
     )
-    (property "Footprint" "LED_THT:LED_D5.0mm" (id 2) (at 129.54 226.06 0)
+    (property "Footprint" "LED_SMD:LED_0805_2012Metric_Pad1.15x1.40mm_HandSolder" (id 2) (at 129.54 226.06 0)
       (effects (font (size 1.27 1.27)) hide)
     )
@@
       (effects (font (size 1.27 1.27)) (justify right))
     )
-    (property "Footprint" "LED_THT:LED_D5.0mm" (id 2) (at 170.18 220.98 0)
+    (property "Footprint" "LED_SMD:LED_0805_2012Metric_Pad1.15x1.40mm_HandSolder" (id 2) (at 170.18 220.98 0)
       (effects (font (size 1.27 1.27)) hide)
     )
@@
       (effects (font (size 1.27 1.27)) (justify left))
     )
-    (property "Footprint" "Capacitor_THT:CP_Radial_D4.0mm_P2.00mm" (id 2) (at 211.7852 328.93 0)
+    (property "Footprint" "Capacitor_SMD:C_0805_2012Metric_Pad1.18x1.45mm_HandSolder" (id 2) (at 211.7852 328.93 0)
       (effects (font (size 1.27 1.27)) hide)
     )
@@
       (effects (font (size 1.27 1.27)) (justify left))
     )
-    (property "Footprint" "Capacitor_THT:CP_Radial_D4.0mm_P2.00mm" (id 2) (at 229.87 243.5352 0)
+    (property "Footprint" "Capacitor_SMD:C_0805_2012Metric_Pad1.18x1.45mm_HandSolder" (id 2) (at 229.87 243.5352 0)
       (effects (font (size 1.27 1.27)) hide)
     )
@@
     )
   )
-  (symbol (lib_id "Connector_Generic:Conn_01x04") (at 43.18 370.84 0) (unit 1)
-    (in_bom yes) (on_board yes)
-    (property "Reference" "J8" (id 0) (at 45.72 370.84 0)
-      (effects (font (size 1.27 1.27)) (justify left))
-    )
-    (property "Value" "OLED_conn" (id 1) (at 45.72 373.38 0)
-      (effects (font (size 1.27 1.27)) (justify left))
-    )
-    (property "Footprint" "Connector_JST:JST_XH_B4B-XH-A_1x04_P2.50mm_Vertical" (id 2) (at 43.18 370.84 0)
-      (effects (font (size 1.27 1.27)) hide)
-    )
-    (property "Datasheet" "~" (id 3) (at 43.18 370.84 0)
-      (effects (font (size 1.27 1.27)) hide)
-    )
-  )
   (symbol (lib_id "Connector_Generic:Conn_01x04") (at 274.32 67.31 0) (mirror x) (unit 1)
     (in_bom yes) (on_board yes)
@@
     )
   )
+  (symbol (lib_id "Connector_Generic:Conn_01x05") (at 43.18 370.84 0) (unit 1)
+    (in_bom yes) (on_board yes)
+    (property "Reference" "J8" (id 0) (at 45.72 369.57 0)
+      (effects (font (size 1.27 1.27)) (justify left))
+    )
+    (property "Value" "OLED_conn" (id 1) (at 45.72 372.11 0)
+      (effects (font (size 1.27 1.27)) (justify left))
+    )
+    (property "Footprint" "Connector_JST:JST_XH_B5B-XH-A_1x05_P2.50mm_Vertical" (id 2) (at 43.18 370.84 0)
+      (effects (font (size 1.27 1.27)) hide)
+    )
+    (property "Datasheet" "~" (id 3) (at 43.18 370.84 0)
+      (effects (font (size 1.27 1.27)) hide)
+    )
+  )
   (symbol (lib_id "Connector_Generic:Conn_01x06") (at 274.32 27.94 0) (unit 1)
     (in_bom yes) (on_board yes)
@@
     )
     (path "/4b2aaea4-045d-4e9f-a942-01b30b3a257c"
-      (reference "C1") (unit 1) (value "100n") (footprint "Capacitor_THT:CP_Radial_D4.0mm_P2.00mm")
+      (reference "C1") (unit 1) (value "100n") (footprint "Capacitor_SMD:C_0805_2012Metric_Pad1.18x1.45mm_HandSolder")
     )
     (path "/f7965251-9827-42d9-8630-9abb56d15421"
-      (reference "C2") (unit 1) (value "100n") (footprint "Capacitor_THT:CP_Radial_D4.0mm_P2.00mm")
+      (reference "C2") (unit 1) (value "100n") (footprint "Capacitor_SMD:C_0805_2012Metric_Pad1.18x1.45mm_HandSolder")
     )
     (path "/f3a504b2-c4ce-43cc-ad77-e0255d46d57c"
-      (reference "D1") (unit 1) (value "LED") (footprint "LED_THT:LED_D5.0mm")
+      (reference "D1") (unit 1) (value "LED") (footprint "LED_SMD:LED_0805_2012Metric_Pad1.15x1.40mm_HandSolder")
     )
     (path "/990170f9-d2c8-408d-aab7-0cb6a1e0931c"
-      (reference "D2") (unit 1) (value "LED Red") (footprint "LED_THT:LED_D5.0mm")
+      (reference "D2") (unit 1) (value "LED Red") (footprint "LED_SMD:LED_0805_2012Metric_Pad1.15x1.40mm_HandSolder")
     )
     (path "/578d094c-6d6d-410f-99be-65ae582c55e7"
@@
       (reference "J7") (unit 1) (value "Fan_conn") (footprint "Connector_JST:JST_XH_B4B-XH-A_1x04_P2.50mm_Vertical")
     )
-    (path "/c5d6cac8-5514-4cb6-8a32-4eb7b3fd13bc"
-      (reference "J8") (unit 1) (value "OLED_conn") (footprint "Connector_JST:JST_XH_B4B-XH-A_1x04_P2.50mm_Vertical")
+    (path "/850f9891-8fab-47d7-afe9-5072797aad05"
+      (reference "J8") (unit 1) (value "OLED_conn") (footprint "Connector_JST:JST_XH_B5B-XH-A_1x05_P2.50mm_Vertical")
     )
     (path "/9f3e25cb-1b33-4910-b92b-80b6c27a3286"
